File: BenchBotv3.0 Electrical System Schematic/BenchBotv3.0 Electrical System Schematic.kicad_sch (KiCad schematic)
At the start: 42 parts, among them J1 2.5mm ID Male Barrel jack, J1 CC I/O-5, J2 CC DI-6, J3 5mm Plug Header, J4 CC PWR, K1 DPDT - 2905660, K2 DPDT - 2905660, K3 SPDT - 52001, K4 OPTO SPDT - 52510, K5 OPTO SPDT - 52510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

Commit message: 75% done with schematic update
Parts:
- removed F1, F2: Fuse, symbol Device:Fuse
- removed F3, F4: 2A Fuse, symbol Device:Fuse
- removed F5: 0.5A Fuse, symbol Device:Fuse
- removed NT1, NT3, NT4: NetTie_2, symbol Device:NetTie_2
- added F10, F6, F7, F8, F9: ~, symbol PSA:Fused_Terminal_Block
- added F11: 0.5A, symbol PSA:Fused_Terminal_Block
- added J10, J11, J12, J13, J14, J15: CC DI-6, symbol Connector:Conn_01x03_Socket
- added J5: CC I/O-4, symbol Connector:Conn_01x03_Socket
- added J6: CC I/O-3, symbol Connector:Conn_01x03_Socket
- added J7: CC I/O-2, symbol Connector:Conn_01x03_Socket
- added J8: CC I/O-1, symbol Connector:Conn_01x03_Socket
- added J9: CC I/O-0, symbol Connector:Conn_01x03_Socket
- renumbered K3 to K1, K4 to K2, K5 to K3, K1 to K4, K2 to K5
Connections:
- net Batt- is gone; now on net GND: C1.1 (Pin_1), GB1.
- net CC GND is gone; now on net GND: K1.A2
- net +BATT: no longer K4.24, PWR1. (GND)
- net Enable Sink (48V-) IN: now also TB7. (Jumper)
- net Enable Sink (48V-) OUT: now also TB9. (Jumper)
- net Enable Source (48V+) IN: now also TB8. (Jumper)
- net Enable Source (48V+) OUT: now also TB10. (Jumper)
- net Flash Power Out 12.6VDC: now also F6.
- net GND: now also K5.A2, PWR2. (GND), PWR3. (GND), TB1., TB10., TB6.
- net SENSE - Enable Sink (48V-): now also TB4. (Jumper), TB5. (Jumper)
- net SENSE - Enable Source (48V+): now also TB6. (Jumper)
- net Z Axis Brake 24V+: now also K4.11, F8.; no longer C11.3 (Pin_3)
- net 24V+: now reaches TB2.
- net 24V+: now also J3.1 (Pin_1), J4.1 (Pin_1), K2.11, K3.11, K4.14, PWR2. (GND), TB1., F10., F11.
- net 48V Batt+ Prot: now reaches TB10.
- net 48V Batt+ Prot: now also CB1.1, K4.24, PWR1. (GND), PWR2. (GND), PWR3. (GND), TB6.
- net at K4.A1: now also K3.14; no longer K3.11
- net PC Barrel+: now reaches PWR3. (GND)
- net PC Barrel+: now also J1.2 (Pin_2); no longer PWR2. (GND)
- net Case Fan 24V+: now reaches M1.1 (+)
- net Case Fan 24V+: now also F11.
- net 48V Batt+: now reaches C1.2 (Pin_2), CB1.2
- removed net 24V BUS: J3.1 (Pin_1), J4.1 (Pin_1), K3.14, K4.14
- new net: TB4. (Jumper), TB5. (Jumper)
- new net 12.6V+: F6., PWR1. (GND)
- new net Z Axis Brake 24V+ Prot: C11.3 (Pin_3), F8.
- no-connect marks 19 -> 21
Other:
- note added: "48 to 19.0V"
- note added: "48 to 24.0V"
- note added: "CC E-Stop Assert Relay"
- note added: "Clear Core Conenctions"
- note added: "Conenct to door GND lug"
- note added: "Cooling Fan"
- note added: "DC-DC Power Supplies"
- note added: "E-Stop Relay System"
- note added: "External Connections"
- note added: "Hardware E-stop Relay"
- note added: "Inside +"
- note added: "Mini PC"
- note added: "Network Switch"
- note added: "Spare Relay"
- note removed: "48 to 19V"
- note removed: "48 to 24V"
- moved on the sheet: C1, C11, C2, C3, C4, C9, CB1, CB2, GB1, GB2, J1, J2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

Commit message: Updated schematic to 85% complete
Parts:
- added J16: PD-P2, symbol Connector:Conn_01x02_Socket
- added J17: PD-P5, symbol Connector:Conn_01x04_Socket
- added J18: PD-P6, symbol Connector:Conn_01x04_Socket
- added J19: PD-P4, symbol Connector:Conn_01x02_Socket
Connections:
- net 48V Batt+ Prot is gone; now on net PWR1 - Vin: CB1.1, K4.24, PWR1. (GND), PWR2. (GND), PWR3. (GND), TB10., TB6.
- net GND: now also J16.2 (Pin_2), J19.2 (Pin_2)
- net NW SW - 1: now reaches TB2.
- net NW SW - 1: now also F10., F11., J3.1 (Pin_1), J4.1 (Pin_1), K3.11, K4.14, PWR2. (GND), TB1., J19.1 (Pin_1)
- net CC DI-6 -1: now reaches K2.14
- net CC DI-6 -1: now also J2.1 (Pin_1)
- net PWR1 - Vin: now reaches TB10.
- net CC DI-6 -3: now reaches J2.3 (Pin_3)
- net CC DI-6 -3: now also K2.11
- removed net 24V+: F10., F11., J3.1 (Pin_1), J4.1 (Pin_1), K2.11, K3.11, K4.14, PWR2. (GND), TB1., TB2.
- net Motor Power renamed Motor Power Prot
- net Motor Power Prot: now also J16.1 (Pin_1)
- new net: TB4. (Jumper), TB5. (Jumper)
- no-connect marks 21 -> 30
Other:
- note added: "ClearPath Power Distribution Board Connections"
- note added: "Internal Equipment Connections"
- note added: "Premade Cable Connections X-Axis Motor"
- note added: "Premade Cable Connections Z-Axis Motor"
- note added: "The wire MAY be color coded for additional wiring guidance, in these cases the color coding represents the prefered color of the physical wire"
- note added: "There may be an additional black label for more information"
- note added: "When a wire ends with a PWR symbol, it is up to the technician to determine the appropriate landing terminal"
- note added: "Wires are labeled as destination and pin # / name"
- moved on the sheet: C11, J1, J10, J11, J12, J13, J14, J15, J2, J4, J5, J6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

Commit message: Updated E-stop Wiring
Connections:
- net NW SW - 1: now also F7.
- net +BATT renamed Aux 24V+ Out
- net Aux 24V+ Out: now also F7.
- new net: TB10. (Jumper), TB6. (Jumper)
- new net: TB4. (Jumper), TB5. (Jumper)
- no-connect marks 30 -> 28
